File: hardware/altcrab_r0.0.1/IO.kicad_sch (KiCad schematic)
At the start: 37 parts, among them J1 Conn_01x12_Male, J2 Conn_01x16_Male, J3 USB_C_Receptacle_USB2.0, SW1 SW_Push, U9 74HC4067BQ

Commit message: update footprint in schematic for feather pins
Parts:
- J1: footprint gkl_conn:Feather_PinHeader_1x12 -> w531t4_altcrab_footprints:Feather_PinHeader_1x12 _ castellated
- J2: footprint gkl_conn:Feather_PinHeader_1x16 -> w531t4_altcrab_footprints:Feather_PinHeader_1x16_castellated
Changed lines of the file:
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@@
 			)
 		)
-		(property "Footprint" "gkl_conn:Feather_PinHeader_1x16"
+		(property "Footprint" "w531t4_altcrab_footprints:Feather_PinHeader_1x16_castellated"
 			(at 229.87 114.3 0)
 			(effects
@@
 			)
 		)
-		(property "Footprint" "gkl_conn:Feather_PinHeader_1x12"
+		(property "Footprint" "w531t4_altcrab_footprints:Feather_PinHeader_1x12 _ castellated"
 			(at 223.52 72.39 0)
 			(effects
